Commit message: gazebo final support, navigation final tweaks, navigation endurance test node and some clean up + readme

File: pioneer_utils/gazebo/pioneer3at.xacro (robot description, xacro)
@@ -70,5 +70,5 @@
 	<joint name="hokuyo_joint" type="fixed">
 		<axis xyz="0 1 0" />
-		<origin xyz="0.2 0 0.4" rpy="0 0 0"/>
+		<origin xyz="-0.19 0 0.4" rpy="0 0 3.141592"/>
 		<parent link="base_link"/>
 		<child link="laser"/>
@@ -99,5 +99,5 @@
 	<joint name="camera_joint" type="fixed">
 		<axis xyz="0 1 0" />
-		<origin xyz="0.2 0 0.47" rpy="0 0 0"/>
+		<origin xyz="-0.04 0 0.40" rpy="0 0 0"/>
 		<parent link="base_link"/>
 		<child link="camera_link"/>
@@ -108,5 +108,5 @@
 			<origin xyz="0 0 0" rpy="0 0 0"/>
 			<geometry>
-				<box size="0.07271 0.27794 0.073"/>
+				<box size="0.07271 0.21 0.073"/>
 			</geometry>
 		</collision>

Commit message: gazebo new meshes and submodules voice and audio

File: pioneer_utils/gazebo/pioneer3at.xacro (robot description, xacro)
@@ -13,4 +13,6 @@
 	<!-- Import xacro:macro for wheels -->
 	<xacro:include filename="$(find pioneer_utils)/gazebo/pioneer3at_wheels.xacro" />
+	<!-- Import xacro:macro for pilars -->
+	<xacro:include filename="$(find pioneer_utils)/gazebo/pioneer3at_pilars.xacro" />
 	<!-- Chassis -->
 	<link name="base_link">
@@ -68,60 +70,152 @@
 		<child link="top_plate"/>
 	</joint>
-	<joint name="hokuyo_joint" type="fixed">
+	<!-- Long pilars -->
+	<xacro:longpilar_front suffix="left" reflect="1"/>
+	<xacro:longpilar_front suffix="right" reflect="-1"/>
+	<!-- Side_left -->
+	<link name="side_plate_left">
+		<inertial>
+			<mass value="0.1"/>
+			<origin xyz="0 0 0"/>
+			<inertia ixx="1.0" ixy="0.0" ixz="0.0"
+				 iyy="1.0" iyz="0.0"
+ 				izz="1.0"/>
+		</inertial>
+		<visual name="side_visual">
+			<origin xyz="0 0 0" rpy="1.57079 0 0"/>
+			<geometry name="pioneer_geom">
+				<mesh filename="package://pioneer_utils/gazebo/meshes/lateral.stl"/>
+			</geometry>
+			<material name="ChassisRed">
+				<color rgba="0.8 0.0 0.0 1.0"/>
+			</material>
+		</visual>
+		<collision>
+			<origin xyz="0 0 0" rpy="1.57079 0 0"/>
+			<geometry>
+				<mesh filename="package://pioneer_utils/gazebo/meshes/lateral.stl"/>
+			</geometry>
+		</collision>
+	</link>
+	<joint name="base_sideleft_joint" type="fixed">
+		<origin xyz="0.02 0.165 0.1" rpy="0 0 0"/>
+		<parent link="top_plate"/>
+		<child link="side_plate_left"/>
+	</joint>
+		<!-- Side_right -->
+	<link name="side_plate_right">
+		<inertial>
+			<mass value="0.1"/>
+			<origin xyz="0 0 0"/>
+			<inertia ixx="1.0" ixy="0.0" ixz="0.0"
+				 iyy="1.0" iyz="0.0"
+ 				izz="1.0"/>
+		</inertial>
+		<visual name="side_visual">
+			<origin xyz="0 0 0" rpy="1.57079 0 0"/>
+			<geometry name="pioneer_geom">
+				<mesh filename="package://pioneer_utils/gazebo/meshes/lateral.stl"/>
+			</geometry>
+			<material name="ChassisRed">
+				<color rgba="0.8 0.0 0.0 1.0"/>
+			</material>
+		</visual>
+		<collision>
+			<origin xyz="0 0 0" rpy="1.57079 0 0"/>
+			<geometry>
+				<mesh filename="package://pioneer_utils/gazebo/meshes/lateral.stl"/>
+			</geometry>
+		</collision>
+	</link>
+	<joint name="base_sideright_joint" type="fixed">
+		<origin xyz="0.02 -0.162 0.1" rpy="0 0 0"/>
+		<parent link="top_plate"/>
+		<child link="side_plate_right"/>
+	</joint>
+	<!-- Top top-->
+	<link name="toptop_plate">
+		<inertial>
+			<mass value="0.1"/>
+			<origin xyz="0 0 0"/>
+			<inertia ixx="1.0" ixy="0.0" ixz="0.0"
+				 iyy="1.0" iyz="0.0"
+ 				izz="1.0"/>
+		</inertial>
+		<visual name="toptop_visual">
+			<origin xyz="0 0 0" rpy="0 0 0"/>
+			<geometry name="pioneer_geom">
+				<mesh filename="package://pioneer_utils/gazebo/meshes/toptop.stl"/>
+			</geometry>
+			<material name="TopBlack">
+					<color rgba="0.038 0.038 0.038 1.0"/>
+			</material>
+		</visual>
+		<collision>
+			<origin xyz="0 0 0" rpy="0 0 0"/>
+			<geometry>
+				<box size="0 0 0"/>
+			</geometry>
+		</collision>
+	</link>
+	<joint name="base_toptop_joint" type="fixed">
+		<origin xyz="0.003 0 0.2" rpy="0 0 0"/>
+		<parent link="top_plate"/>
+		<child link="toptop_plate"/>
+	</joint>
+	<!-- Sick Laser -->
+	<link name="laser">
+		<collision>
+			<origin xyz="0 0 -0.06" rpy="0 0 0"/>
+			<geometry>
+				<box size="0.1 0.1 0.16"/>
+			</geometry>
+		</collision>
+		<visual>
+			<origin xyz="0 0 -0.06" rpy="3.141592 0 0"/>
+			<geometry>
+				<mesh filename="package://pioneer_utils/gazebo/meshes/sick_lms100.dae"/>
+			</geometry>
+		</visual>
+		<inertial>
+			<mass value="1e-5" />
+			<inertia ixx="1e-6" ixy="0" ixz="0" iyy="1e-6" iyz="0" izz="1e-6" />
+		</inertial>
+	</link>
+	<joint name="laser_joint" type="fixed">
 		<axis xyz="0 1 0" />
-		<origin xyz="-0.19 0 0.4" rpy="0 0 3.141592"/>
+		<origin xyz="-0.195 0 0.4" rpy="0 0 3.141592"/>
 		<parent link="base_link"/>
 		<child link="laser"/>
 	</joint>
-	<!-- Hokuyo Laser -->
-	<link name="laser">
-		<collision>
-			<origin xyz="0 0 0" rpy="0 0 0"/>
-			<geometry>
-				<box size="0.1 0.1 0.16"/>
-			</geometry>
-		</collision>
-		<visual>
-			<origin xyz="0 0 -0.06" rpy="3.141592 0 0"/>
-			<geometry>
-				<mesh filename="package://pioneer_utils/gazebo/meshes/sick_lms100.dae"/>
-			</geometry>
-		</visual>
-		<inertial>
-			<mass value="1e-5" />
-			<inertia ixx="1e-6" ixy="0" ixz="0" iyy="1e-6" iyz="0" izz="1e-6" />
-		</inertial>
-	</link>
+	<!-- Wheels, axes and hubs -->
 	<xacro:p3at_front suffix="left" reflect="1"/>
 	<xacro:p3at_front suffix="right" reflect="-1"/>
-	<xacro:p3at_back suffix="left" reflect="1"/>
-	<xacro:p3at_back suffix="right" reflect="-1"/>
+	<!-- Camera -->
+	<link name="camera_link">
+		<collision>
+			<origin xyz="0 0 0" rpy="0 0 0"/>
+			<geometry>
+				<box size="0.06 0.21 0.070"/>
+			</geometry>
+		</collision>
+		<visual>
+			<origin xyz="0 0 -0.01" rpy="0 0 1.570796"/>
+			<geometry>
+				<mesh filename="package://pioneer_utils/gazebo/meshes/kinect.dae"/>
+			</geometry>
+		</visual>
+		<inertial>
+			<mass value="0.546" />
+			<origin xyz="0 0 0" rpy="0 0 0"/>
+			<inertia ixx="0.003881243" ixy="0" ixz="0" iyy="0.000498940" iyz="0" izz="0.003879257" />
+		</inertial>
+	</link>
 	<joint name="camera_joint" type="fixed">
 		<axis xyz="0 1 0" />
-		<origin xyz="-0.04 0 0.40" rpy="0 0 0"/>
-		<parent link="base_link"/>
+		<origin xyz="0 0 0.10" rpy="0 0 0"/>
+		<parent link="top_plate"/>
 		<child link="camera_link"/>
 	</joint>
-	<!-- Camera -->
-	<link name="camera_link">
-		<collision>
-			<origin xyz="0 0 0" rpy="0 0 0"/>
-			<geometry>
-				<box size="0.07271 0.21 0.073"/>
-			</geometry>
-		</collision>
-		<visual>
-			<origin xyz="0 0 -0.01" rpy="0 0 1.570796"/>
-			<geometry>
-				<mesh filename="package://pioneer_utils/gazebo/meshes/kinect.dae"/>
-			</geometry>
-		</visual>
-		<inertial>
-			<mass value="0.546" />
-			<origin xyz="0 0 0" rpy="0 0 0"/>
-			<inertia ixx="0.003881243" ixy="0" ixz="0" iyy="0.000498940" iyz="0" izz="0.003879257" />
-		</inertial>
-	</link>
-<!-- from turtlebot!! -->
+<!-- camera config from turtlebot!! -->
 	<joint name="camera_rgb_joint" type="fixed">
 		<origin xyz="-0.087 -0.0125 0.2870" rpy="0 0 0"/>

Commit message: mesh and freecad parts, hardware statis transforms adapted to new status, navigation w/o map

File: pioneer_utils/gazebo/pioneer3at.xacro (robot description, xacro)
@@ -99,5 +99,5 @@
 	</link>
 	<joint name="base_sideleft_joint" type="fixed">
-		<origin xyz="0.02 0.165 0.1" rpy="0 0 0"/>
+		<origin xyz="0.018 0.165 0.1" rpy="0 0 0"/>
 		<parent link="top_plate"/>
 		<child link="side_plate_left"/>
@@ -129,5 +129,5 @@
 	</link>
 	<joint name="base_sideright_joint" type="fixed">
-		<origin xyz="0.02 -0.162 0.1" rpy="0 0 0"/>
+		<origin xyz="0.018 -0.162 0.1" rpy="0 0 0"/>
 		<parent link="top_plate"/>
 		<child link="side_plate_right"/>

Commit message: navigation voxel layers, gazebo mesh model, still problems on gazebo local nav

File: pioneer_utils/gazebo/pioneer3at.xacro (robot description, xacro)
@@ -99,5 +99,5 @@
 	</link>
 	<joint name="base_sideleft_joint" type="fixed">
-		<origin xyz="0.018 0.165 0.1" rpy="0 0 0"/>
+		<origin xyz="-0.02 0.165 0.1" rpy="0 0 0"/>
 		<parent link="top_plate"/>
 		<child link="side_plate_left"/>
@@ -129,7 +129,157 @@
 	</link>
 	<joint name="base_sideright_joint" type="fixed">
-		<origin xyz="0.018 -0.162 0.1" rpy="0 0 0"/>
+		<origin xyz="-0.02 -0.162 0.1" rpy="0 0 0"/>
 		<parent link="top_plate"/>
 		<child link="side_plate_right"/>
+	</joint>
+		<!-- Side_back_down_right -->
+	<link name="side_plate_back_down_right">
+		<inertial>
+			<mass value="0.1"/>
+			<origin xyz="0 0 0"/>
+			<inertia ixx="1.0" ixy="0.0" ixz="0.0"
+				 iyy="1.0" iyz="0.0"
+ 				izz="1.0"/>
+		</inertial>
+		<visual name="side_visual">
+			<origin xyz="0 0 0" rpy="0 0 0"/>
+			<geometry name="pioneer_geom">
+				<box size="0.15 0.003 0.11"/>
+			</geometry>
+			<material name="ChassisRed">
+				<color rgba="0.8 0.0 0.0 1.0"/>
+			</material>
+		</visual>
+		<collision>
+			<origin xyz="0 0 0" rpy="0 0 0"/>
+			<geometry>
+				<box size="0.15 0.003 0.11"/>
+			</geometry>
+		</collision>
+	</link>
+	<joint name="base_sidebackdownright_joint" type="fixed">
+		<origin xyz="-0.205 -0.095 0.055" rpy="0 0 -1.1"/>
+		<parent link="top_plate"/>
+		<child link="side_plate_back_down_right"/>
+	</joint>
+		<!-- Side_back_up_right -->
+	<link name="side_plate_back_up_right">
+		<inertial>
+			<mass value="0.1"/>
+			<origin xyz="0 0 0"/>
+			<inertia ixx="1.0" ixy="0.0" ixz="0.0"
+				 iyy="1.0" iyz="0.0"
+ 				izz="1.0"/>
+		</inertial>
+		<visual name="side_visual">
+			<origin xyz="0 0 0" rpy="0 0 0"/>
+			<geometry name="pioneer_geom">
+				<box size="0.15 0.003 0.08"/>
+			</geometry>
+			<material name="ChassisRed">
+				<color rgba="0.8 0.0 0.0 1.0"/>
+			</material>
+		</visual>
+		<collision>
+			<origin xyz="0 0 0" rpy="0 0 0"/>
+			<geometry>
+				<box size="0.15 0.003 0.08"/>
+			</geometry>
+		</collision>
+	</link>
+	<joint name="base_sidebackupright_joint" type="fixed">
+		<origin xyz="-0.205 -0.095 0.16" rpy="0 0 -1.1"/>
+		<parent link="top_plate"/>
+		<child link="side_plate_back_up_right"/>
+	</joint>
+		<!-- Side_back_down_left -->
+	<link name="side_plate_back_down_left">
+		<inertial>
+			<mass value="0.1"/>
+			<origin xyz="0 0 0"/>
+			<inertia ixx="1.0" ixy="0.0" ixz="0.0"
+				 iyy="1.0" iyz="0.0"
+ 				izz="1.0"/>
+		</inertial>
+		<visual name="side_visual">
+			<origin xyz="0 0 0" rpy="0 0 0"/>
+			<geometry name="pioneer_geom">
+				<box size="0.15 0.003 0.11"/>
+			</geometry>
+			<material name="ChassisRed">
+				<color rgba="0.8 0.0 0.0 1.0"/>
+			</material>
+		</visual>
+		<collision>
+			<origin xyz="0 0 0" rpy="0 0 0"/>
+			<geometry>
+				<box size="0.15 0.003 0.11"/>
+			</geometry>
+		</collision>
+	</link>
+	<joint name="base_sidebackdownleft_joint" type="fixed">
+		<origin xyz="-0.205 0.095 0.055" rpy="0 0 1.1"/>
+		<parent link="top_plate"/>
+		<child link="side_plate_back_down_left"/>
+	</joint>
+		<!-- Side_back_up_left -->
+	<link name="side_plate_back_up_left">
+		<inertial>
+			<mass value="0.1"/>
+			<origin xyz="0 0 0"/>
+			<inertia ixx="1.0" ixy="0.0" ixz="0.0"
+				 iyy="1.0" iyz="0.0"
+ 				izz="1.0"/>
+		</inertial>
+		<visual name="side_visual">
+			<origin xyz="0 0 0" rpy="0 0 0"/>
+			<geometry name="pioneer_geom">
+				<box size="0.15 0.003 0.08"/>
+			</geometry>
+			<material name="ChassisRed">
+				<color rgba="0.8 0.0 0.0 1.0"/>
+			</material>
+		</visual>
+		<collision>
+			<origin xyz="0 0 0" rpy="0 0 0"/>
+			<geometry>
+				<box size="0.15 0.003 0.08"/>
+			</geometry>
+		</collision>
+	</link>
+	<joint name="base_sidebackupleft_joint" type="fixed">
+		<origin xyz="-0.205 0.095 0.16" rpy="0 0 1.1"/>
+		<parent link="top_plate"/>
+		<child link="side_plate_back_up_left"/>
+	</joint>
+		<!-- Side_back_up -->
+	<link name="side_plate_back_up">
+		<inertial>
+			<mass value="0.1"/>
+			<origin xyz="0 0 0"/>
+			<inertia ixx="1.0" ixy="0.0" ixz="0.0"
+				 iyy="1.0" iyz="0.0"
+ 				izz="1.0"/>
+		</inertial>
+		<visual name="side_visual">
+			<origin xyz="0 0 0" rpy="0 0 0"/>
+			<geometry name="pioneer_geom">
+				<box size="0.058 0.003 0.05"/>
+			</geometry>
+			<material name="ChassisRed">
+				<color rgba="0.8 0.0 0.0 1.0"/>
+			</material>
+		</visual>
+		<collision>
+			<origin xyz="0 0 0" rpy="0 0 0"/>
+			<geometry>
+				<box size="0.058 0.003 0.05"/>
+			</geometry>
+		</collision>
+	</link>
+	<joint name="base_sidebackup_joint" type="fixed">
+		<origin xyz="-0.24 0. 0.175" rpy="0 0 1.57079"/>
+		<parent link="top_plate"/>
+		<child link="side_plate_back_up"/>
 	</joint>
 	<!-- Top top-->
@@ -172,5 +322,5 @@
 		</collision>
 		<visual>
-			<origin xyz="0 0 -0.06" rpy="3.141592 0 0"/>
+			<origin xyz="0 0 -0.05" rpy="3.141592 0 0"/>
 			<geometry>
 				<mesh filename="package://pioneer_utils/gazebo/meshes/sick_lms100.dae"/>
@@ -184,5 +334,5 @@
 	<joint name="laser_joint" type="fixed">
 		<axis xyz="0 1 0" />
-		<origin xyz="-0.195 0 0.4" rpy="0 0 3.141592"/>
+		<origin xyz="-0.195 0 0.39" rpy="0 0 3.141592"/>
 		<parent link="base_link"/>
 		<child link="laser"/>
